File: hardware/QAZ_65/pcb/QAZ_65/QAZ_65_externals.sch (KiCad schematic (older format))
At the start: 6 parts, among them CN1 USB2.0_TYPE_C, J1 1x6 2.54mm

Commit message: QAZ 65% v1.1: updating from v1.0
closes #5
closes #3

QAZ 65% v1.1:

 - Switch for BOOT (PG for booting into bootloader tor ProGram the
   board, KB for booting into KeyBoard)
 - New RGB driver IC, which allows driving RGB LEDS in a grid format
Parts:
- removed J1: 1x6 2.54mm, Connector_PinHeader_2.54mm:PinHeader_1x06_P2.54mm_Horizontal, symbol Connector_Generic:Conn_01x06
- removed R15, R16: 10k, Resistor_SMD:R_0603_1608Metric_Pad1.05x0.95mm_HandSolder, symbol Device:R_Small_US
- renumbered R17 to R15
Other:
- note removed: "SWD/Serial Debugger Header"
Changed lines of the file:
@@
 EESchema Schematic File Version 4
-LIBS:QAZ_65-cache
 EELAYER 30 0
 EELAYER END
 $Descr A4 11693 8268
 encoding utf-8
-Sheet 3 3
+Sheet 2 4
 Title "QAZ 65% External"
-Date "2020-12-23"
+Date "2021-05-11"
 Rev "v1.1"
 Comp "Anthony Needles"
@@
 Comment4 ""
 $EndDescr
-$Comp
-L power:+3.3V #PWR?
-U 1 1 5F98A26F
-P 5800 2650
-AR Path="/5F98A26F" Ref="#PWR?"  Part="1"
-AR Path="/5F96C310/5F98A26F" Ref="#PWR036"  Part="1"
-F 0 "#PWR036" H 5800 2500 50  0001 C CNN
-F 1 "+3.3V" H 5800 2800 50  0000 C CNN
-F 2 "" H 5800 2650 50  0001 C CNN
-F 3 "" H 5800 2650 50  0001 C CNN
-	1    5800 2650
-	1    0    0    -1
-$EndComp
-$Comp
-L Device:R_Small_US R?
-U 1 1 5F98A28C
-P 5700 3550
-AR Path="/5F98A28C" Ref="R?"  Part="1"
-AR Path="/5F96C310/5F98A28C" Ref="R16"  Part="1"
-F 0 "R16" H 5900 3500 50  0000 R CNN
-F 1 "10k" H 5900 3600 50  0000 R CNN
-F 2 "Resistor_SMD:R_0603_1608Metric_Pad1.05x0.95mm_HandSolder" H 5700 3550 50  0001 C CNN
-F 3 "~" H 5700 3550 50  0001 C CNN
-	1    5700 3550
-	-1   0    0    1
-$EndComp
-$Comp
-L Device:R_Small_US R?
-U 1 1 5F98A292
-P 5600 2750
-AR Path="/5F98A292" Ref="R?"  Part="1"
-AR Path="/5F96C310/5F98A292" Ref="R15"  Part="1"
-F 0 "R15" H 5800 2700 50  0000 R CNN
-F 1 "10k" H 5800 2800 50  0000 R CNN
-F 2 "Resistor_SMD:R_0603_1608Metric_Pad1.05x0.95mm_HandSolder" H 5600 2750 50  0001 C CNN
-F 3 "~" H 5600 2750 50  0001 C CNN
-	1    5600 2750
-	-1   0    0    1
-$EndComp
-$Comp
-L power:+3.3V #PWR?
-U 1 1 5F98A299
-P 5600 2650
-AR Path="/5F98A299" Ref="#PWR?"  Part="1"
-AR Path="/5F96C310/5F98A299" Ref="#PWR033"  Part="1"
-F 0 "#PWR033" H 5600 2500 50  0001 C CNN
-F 1 "+3.3V" H 5550 2800 50  0000 C CNN
-F 2 "" H 5600 2650 50  0001 C CNN
-F 3 "" H 5600 2650 50  0001 C CNN
-	1    5600 2650
-	1    0    0    -1
-$EndComp
-Text Notes 4900 2400 0    50   ~ 0
-SWD/Serial Debugger Header
 $Comp
 L QAZ:USB2.0_TYPE_C CN?
@@
 P 5050 4750
 AR Path="/5F98A2C9" Ref="#PWR?"  Part="1"
-AR Path="/5F96C310/5F98A2C9" Ref="#PWR032"  Part="1"
-F 0 "#PWR032" H 5050 4600 50  0001 C CNN
+AR Path="/5F96C310/5F98A2C9" Ref="#PWR024"  Part="1"
+F 0 "#PWR024" H 5050 4600 50  0001 C CNN
 F 1 "+5V" H 5065 4923 50  0000 C CNN
 F 2 "" H 5050 4750 50  0001 C CNN
@@
 P 6450 4750
 AR Path="/5F98A2D1" Ref="#PWR?"  Part="1"
-AR Path="/5F96C310/5F98A2D1" Ref="#PWR038"  Part="1"
-F 0 "#PWR038" H 6450 4600 50  0001 C CNN
+AR Path="/5F96C310/5F98A2D1" Ref="#PWR026"  Part="1"
+F 0 "#PWR026" H 6450 4600 50  0001 C CNN
 F 1 "+5V" H 6465 4923 50  0000 C CNN
 F 2 "" H 6450 4750 50  0001 C CNN
@@
 P 5750 5700
 AR Path="/5F98A2F4" Ref="#PWR?"  Part="1"
-AR Path="/5F96C310/5F98A2F4" Ref="#PWR035"  Part="1"
-F 0 "#PWR035" H 5750 5450 50  0001 C CNN
+AR Path="/5F96C310/5F98A2F4" Ref="#PWR025"  Part="1"
+F 0 "#PWR025" H 5750 5450 50  0001 C CNN
 F 1 "GND" H 5755 5527 50  0001 C CNN
 F 2 "" H 5750 5700 50  0001 C CNN
@@
 P 4950 5450
 AR Path="/5F98A302" Ref="#PWR?"  Part="1"
-AR Path="/5F96C310/5F98A302" Ref="#PWR031"  Part="1"
-F 0 "#PWR031" H 4950 5200 50  0001 C CNN
+AR Path="/5F96C310/5F98A302" Ref="#PWR023"  Part="1"
+F 0 "#PWR023" H 4950 5200 50  0001 C CNN
 F 1 "GND" H 4955 5277 50  0001 C CNN
 F 2 "" H 4950 5450 50  0001 C CNN
@@
 P 6550 5350
 AR Path="/5F98A30A" Ref="R?"  Part="1"
-AR Path="/5F96C310/5F98A30A" Ref="R17"  Part="1"
-F 0 "R17" H 6700 5300 50  0000 R CNN
+AR Path="/5F96C310/5F98A30A" Ref="R15"  Part="1"
+F 0 "R15" H 6700 5300 50  0000 R CNN
 F 1 "5.1k" H 6800 5400 50  0000 R CNN
 F 2 "Resistor_SMD:R_0603_1608Metric_Pad1.05x0.95mm_HandSolder" H 6550 5350 50  0001 C CNN
@@
 P 6550 5450
 AR Path="/5F98A311" Ref="#PWR?"  Part="1"
-AR Path="/5F96C310/5F98A311" Ref="#PWR039"  Part="1"
-F 0 "#PWR039" H 6550 5200 50  0001 C CNN
+AR Path="/5F96C310/5F98A311" Ref="#PWR027"  Part="1"
+F 0 "#PWR027" H 6550 5200 50  0001 C CNN
 F 1 "GND" H 6555 5277 50  0001 C CNN
 F 2 "" H 6550 5450 50  0001 C CNN
@@
 Wire Notes Line
 	4650 4350 6850 4350
-Text HLabel 5550 3100 0    50   Input ~ 0
-DBG_TX
-Text HLabel 5550 3000 0    50   Output ~ 0
-SWDIO
-Text HLabel 5550 3400 0    50   Output ~ 0
-nRESET
-Wire Wire Line
-	5900 3200 5800 3200
-Wire Wire Line
-	5900 2900 5700 2900
-Text HLabel 5550 2900 0    50   BiDi ~ 0
-SWCLK
-Wire Notes Line
-	6600 3850 4850 3850
-Wire Notes Line
-	4850 2400 6600 2400
 Wire Wire Line
 	6250 4950 6450 4950
@@
 Wire Notes Line
 	6850 4350 6850 5900
-$Comp
-L Connector_Generic:Conn_01x06 J1
-U 1 1 603DD2B3
-P 6100 3100
-F 0 "J1" H 6180 3092 50  0000 L CNN
-F 1 "1x6 2.54mm" H 5900 2700 50  0000 L CNN
-F 2 "Connector_PinHeader_2.54mm:PinHeader_1x06_P2.54mm_Horizontal" H 6100 3100 50  0001 C CNN
-F 3 "~" H 6100 3100 50  0001 C CNN
-	1    6100 3100
-	1    0    0    -1
-$EndComp
-Wire Wire Line
-	5900 3300 5800 3300
-$Comp
-L power:GND #PWR?
-U 1 1 603F090B
-P 5800 3650
-AR Path="/603F090B" Ref="#PWR?"  Part="1"
-AR Path="/5F96C310/603F090B" Ref="#PWR037"  Part="1"
-F 0 "#PWR037" H 5800 3400 50  0001 C CNN
-F 1 "GND" H 5805 3477 50  0001 C CNN
-F 2 "" H 5800 3650 50  0001 C CNN
-F 3 "" H 5800 3650 50  0001 C CNN
-	1    5800 3650
-	1    0    0    -1
-$EndComp
-$Comp
-L power:GND #PWR?
-U 1 1 603F0CED
-P 5700 3650
-AR Path="/603F0CED" Ref="#PWR?"  Part="1"
-AR Path="/5F96C310/603F0CED" Ref="#PWR034"  Part="1"
-F 0 "#PWR034" H 5700 3400 50  0001 C CNN
-F 1 "GND" H 5705 3477 50  0001 C CNN
-F 2 "" H 5700 3650 50  0001 C CNN
-F 3 "" H 5700 3650 50  0001 C CNN
-	1    5700 3650
-	1    0    0    -1
-$EndComp
-Wire Wire Line
-	5800 2650 5800 3200
-Wire Wire Line
-	5700 2900 5700 3450
-Wire Wire Line
-	5600 2850 5600 3000
-Wire Wire Line
-	5600 3000 5900 3000
-Wire Wire Line
-	5800 3300 5800 3650
-Wire Wire Line
-	5900 3400 5550 3400
-Wire Wire Line
-	5550 3100 5900 3100
-Wire Wire Line
-	5600 3000 5550 3000
-Connection ~ 5600 3000
-Wire Wire Line
-	5700 2900 5550 2900
-Connection ~ 5700 2900
-Wire Notes Line
-	6600 2400 6600 3850
-Wire Notes Line
-	4850 2400 4850 3850
 $EndSCHEMATC
