File: hardware/QAZ_65/pcb/QAZ_65/QAZ_65_keys.sch (KiCad schematic (older format))
At the start: 136 parts, among them SW10 Cherry MX, SW11 Cherry MX, SW12 Cherry MX, SW13 Cherry MX, SW14 Cherry MX, SW15 Cherry MX, SW16 Cherry MX, SW17 Cherry MX, SW18 Cherry MX, SW19 Cherry MX, SW2 Cherry MX, SW20 Cherry MX, SW21 Cherry MX, SW22 Cherry MX, SW23 Cherry MX, SW24 Cherry MX, SW25 Cherry MX, SW26 Cherry MX, SW27 Cherry MX, SW28 Cherry MX, SW29 Cherry MX, SW3 Cherry MX, SW30 Cherry MX, SW31 Cherry MX, SW32 Cherry MX, SW33 Cherry MX, SW34 Cherry MX, SW35 Cherry MX, SW36 Cherry MX, SW37 Cherry MX, SW38 Cherry MX, SW39 Cherry MX, SW4 Cherry MX, SW40 Cherry MX, SW41 Cherry MX, SW42 Cherry MX, SW43 Cherry MX, SW44 Cherry MX, SW45 Cherry MX, SW46 Cherry MX, SW47 Cherry MX, SW48 Cherry MX, SW49 Cherry MX, SW5 Cherry MX, SW50 Cherry MX, SW51 Cherry MX, SW52 Cherry MX, SW53 Cherry MX, SW54 Cherry MX, SW55 Cherry MX, SW56 Cherry MX, SW57 Cherry MX, SW58 Cherry MX, SW59 Cherry MX, SW6 Cherry MX, SW60 Cherry MX, SW61 Cherry MX, SW62 Cherry MX, SW63 Cherry MX, SW64 Cherry MX, SW65 Cherry MX, SW66 Cherry MX, SW67 Cherry MX, SW68 Cherry MX, SW69 Cherry MX, SW7 Cherry MX, SW8 Cherry MX, SW9 Cherry MX

Commit message: QAZ 65% v1.1: updating from v1.0
closes #5
closes #3

QAZ 65% v1.1:

 - Switch for BOOT (PG for booting into bootloader tor ProGram the
   board, KB for booting into KeyBoard)
 - New RGB driver IC, which allows driving RGB LEDS in a grid format
Parts:
- renumbered D7 to D10, D8 to D11, D9 to D12, D10 to D13, D11 to D14, D12 to D15, D13 to D16, D14 to D17, D15 to D18, D16 to D19, D17 to D20, D18 to D21, D19 to D22, D20 to D23, D21 to D24, D22 to D25, D23 to D26, D24 to D27, D25 to D28, D26 to D29, D27 to D30, D28 to D31, D29 to D32, D30 to D33, D31 to D34, D32 to D35, D33 to D36, D34 to D37, D35 to D38, D36 to D39, D1 to D4, D37 to D40, D38 to D41, D39 to D42, D40 to D43, D41 to D44, D42 to D45, D43 to D46, D44 to D47, D45 to D48, D46 to D49, D2 to D5, D47 to D50, D48 to D51, D49 to D52, D50 to D53, D51 to D54, D52 to D55, D53 to D56, D54 to D57, D55 to D58, D56 to D59, D3 to D6, D57 to D60, D58 to D61, D59 to D62, D60 to D63, D61 to D64, D62 to D65, D63 to D66, D64 to D67, D65 to D68, D66 to D69, D4 to D7, D67 to D70, D68 to D71, D5 to D8, D6 to D9
