File: hardware/QAZ_65/pcb/QAZ_65/QAZ_65.kicad_pcb (KiCad board)
At the start: 2 copper layers, 309 x 106.5 mm, 245 parts, among them CN1 USB2.0_TYPE_C, J1 1x6 2.54mm, SW1 PTS525, SW10 Cherry MX, SW11 Cherry MX, SW12 Cherry MX, SW13 Cherry MX, SW14 Cherry MX, SW15 Cherry MX, SW16 Cherry MX, SW17 Cherry MX, SW18 Cherry MX, SW19 Cherry MX, SW2 Cherry MX, SW20 Cherry MX, SW21 Cherry MX, SW22 Cherry MX, SW23 Cherry MX, SW24 Cherry MX, SW25 Cherry MX, SW26 Cherry MX, SW27 Cherry MX, SW28 Cherry MX, SW29 Cherry MX, SW3 Cherry MX, SW30 Cherry MX, SW31 Cherry MX, SW32 Cherry MX, SW33 Cherry MX, SW34 Cherry MX, SW35 Cherry MX, SW36 Cherry MX, SW37 Cherry MX, SW38 Cherry MX, SW39 Cherry MX, SW4 Cherry MX, SW40 Cherry MX, SW41 Cherry MX, SW42 Cherry MX, SW43 Cherry MX, SW44 Cherry MX, SW45 Cherry MX, SW46 Cherry MX, SW47 Cherry MX, SW48 Cherry MX, SW49 Cherry MX, SW5 Cherry MX, SW50 Cherry MX, SW51 Cherry MX, SW52 Cherry MX, SW53 Cherry MX, SW54 Cherry MX, SW55 Cherry MX, SW56 Cherry MX, SW57 Cherry MX, SW58 Cherry MX, SW59 Cherry MX, SW6 Cherry MX, SW60 Cherry MX, SW61 Cherry MX, SW62 Cherry MX, SW63 Cherry MX, SW64 Cherry MX, SW65 Cherry MX, SW66 Cherry MX, SW67 Cherry MX, SW68 Cherry MX, SW69 Cherry MX, SW7 Cherry MX, SW8 Cherry MX, SW9 Cherry MX, U1 AP2112K-3.3, U2 STM32F042C6Tx, U3 LP5009RUKR, Y1 8.0000MHz

Commit message: qaz v1.1: fixes going from v1.0->v1.1
Changed from individual pull up/down on BOOT0 MCU pin to switch that can
easily change from one to the other (without soldering). This is
required for programming over USB DFU.

Fixed RESET switch, pins were flipped on part layout.
Parts:
- removed R1: 10k, Resistor_SMD:R_0603_1608Metric_Pad1.05x0.95mm_HandSolder
- removed TP9: TestPoint, QAZ:TestPoint_Thruhole_1.0mm
- added SW70: JS102011SCQN, QAZ:JS102011SCQN_SPDT, F.Cu at (195.9, 161.2)
- moved R2 7.37 mm to (199.4, 169.9)
- moved C2 2.22 mm to (191.4, 167.7)
- moved C4 2.22 mm to (191.4, 169.7)
- moved SB2 2.22 mm to (191.4, 171.2)
- moved R5 0.70 mm to (202.3, 171.4)
Connections:
- R2 pad 1: GND -> Net-(R2-Pad1)
Routing:
- net +3V3: track 247.8 -> 259.2 mm, vias 0 -> 2
- net /COL08: track 61.8 -> 72.8 mm
- net /BOOT0: track 20.2 -> 10.9 mm, vias 0 -> 2
- net Net-(R2-Pad1): track 0.00 -> 6.90 mm
- net Net-(C1-Pad2): track 5.80 -> 10.0 mm
- net /COL12: track 142.5 -> 144.7 mm
- net +5V: track 392.9 -> 390.8 mm
- net /SWCLK: track 128.5 -> 130.6 mm
- net /QAZ Testboard Keys/ROW02: track 324.4 -> 326.2 mm
- net /HB_LED: track 34.3 -> 32.6 mm
- net /QAZ Testboard Keys/ROW04: track 348.6 -> 349.4 mm
- net (no net): track 0.00 -> 0.69 mm
- net /COL07: track 24.2 -> 24.8 mm
- net /ROW02: track 4.01 -> 3.49 mm
Other:
- board text added: "APP"
- board text added: "BOOT"
- board text added: "QAZ 65% v1.1 - Anthony Needles"
- board text removed: "QAZ 65% v1.0 - Anthony Needles"

Commit message: logo: added new qaz logo to doxygen
Also updated Doxyfile with relative paths and started tracking the doc
folder (with media subfolder). The doxygen subfolder is where the
doxygen output goes (and is untracked).

Also created silkscreen component from the logo and added to PCB
Parts:
- added G***: LOGO, QAZ:qaz_logo_20mm, F.Cu at (359.6, 137.4)

Commit message: QAZ 65% v1.1: updating from v1.0
closes #5
closes #3

QAZ 65% v1.1:

 - Switch for BOOT (PG for booting into bootloader tor ProGram the
   board, KB for booting into KeyBoard)
 - New RGB driver IC, which allows driving RGB LEDS in a grid format
Parts:
- removed the C2 at (191.4, 167.7)
- removed the C4 at (191.4, 169.7)
- removed the C8 at (228.6, 178.7)
- removed the D39 at (179.7, 140.7)
- removed J1: 1x6 2.54mm, Connector_PinHeader_2.54mm:PinHeader_1x06_P2.54mm_Horizontal
- removed LED1: RGB0, LED_SMD:LED_RGB_PLCC-6
- removed LED2: RGB1, LED_SMD:LED_RGB_PLCC-6
- removed LED3: RGB2, LED_SMD:LED_RGB_PLCC-6
- removed LED4: BLUE, Resistor_SMD:R_0603_1608Metric_Pad1.05x0.95mm_HandSolder
- removed the R12 at (258.8, 183.2)
- removed the R14 at (214.2, 91.2)
- removed the R4 at (220.4, 171.2)
- removed the REF** at (321.4, 147.4)
- removed the REF** at (278.4, 127.2)
- removed the REF** at (226.4, 147.4)
- removed the REF** at (183.4, 127.2)
- removed the REF** at (126.6, 147.4)
- removed the REF** at (104.4, 127.2)
- removed the SB1 at (242.5, 176.3)
- removed the SB11 at (108.6, 125.9)
- removed the SB19 at (216.6, 161.4)
- removed SB24, SB25, SB26, SB27, SB28, SB29, SB30, SB31, SB32, SB33, SB34, SB35, SB36, SB37, SB38, SB39, SB40, SB41, SB42: SolderBridge, Resistor_SMD:R_0603_1608Metric_Pad1.05x0.95mm_HandSolder
- removed the SB3 at (306.8, 127.7)
- removed the SB4 at (207.4, 127.7)
- removed the SB6 at (220.6, 178.7)
- removed SW70: JS102011SCQN, QAZ:JS102011SCQN_SPDT
- removed the TP13 at (212.1, 163.9)
- removed TP16, TP17, TP18: TestPoint, QAZ:TestPoint_Thruhole_1.0mm
- removed the TP4 at (236.4, 108.7)
- removed the TP7 at (173.9, 175.7)
- added C11: 0.1uF, Capacitor_SMD:C_0603_1608Metric_Pad1.05x0.95mm_HandSolder, F.Cu at (206.1, 170.1)
- added C14: 1uF, Capacitor_SMD:C_0603_1608Metric_Pad1.05x0.95mm_HandSolder, F.Cu at (233.2, 170.7)
- added C3: 1uF, Capacitor_SMD:C_0603_1608Metric_Pad1.05x0.95mm_HandSolder, F.Cu at (190.5, 172.0)
- added C6: 16pF, Capacitor_SMD:C_0603_1608Metric_Pad1.05x0.95mm_HandSolder, F.Cu at (273.6, 182.5)
- added D1: BLUE, Resistor_SMD:R_0603_1608Metric_Pad1.05x0.95mm_HandSolder, F.Cu at (179.8, 173.6)
- added D42: 1N4148, Diode_THT:D_DO-35_SOD27_P7.62mm_Horizontal, F.Cu at (179.7, 137.2)
- added D72: LED_RABG, LED_THT:LED_D5.0mm-4_RGB, F.Cu at (76.9, 165.9)
- added D73: LED_RABG, LED_THT:LED_D5.0mm-4_RGB, F.Cu at (131.2, 165.6)
- added D74: LED_RABG, LED_THT:LED_D5.0mm-4_RGB, F.Cu at (177.3, 165.7)
- added D75: LED_RABG, LED_THT:LED_D5.0mm-4_RGB, F.Cu at (233.8, 162.0)
- added D76: LED_RABG, LED_THT:LED_D5.0mm-4_RGB, F.Cu at (285.3, 165.7)
- added D77: LED_RABG, LED_THT:LED_D5.0mm-4_RGB, F.Cu at (336.1, 165.9)
- added D78: LED_RABG, LED_THT:LED_D5.0mm-4_RGB, F.Cu at (76.9, 137.4)
- added D79: LED_RABG, LED_THT:LED_D5.0mm-4_RGB, F.Cu at (131.2, 130.3)
- added D80: LED_RABG, LED_THT:LED_D5.0mm-4_RGB, F.Cu at (177.3, 141.8)
- added D81: LED_RABG, LED_THT:LED_D5.0mm-4_RGB, F.Cu at (233.8, 130.2)
- added D82: LED_RABG, LED_THT:LED_D5.0mm-4_RGB, F.Cu at (285.3, 141.8)
- added D83: LED_RABG, LED_THT:LED_D5.0mm-4_RGB, F.Cu at (336.0, 137.2)
- added D84: LED_RABG, LED_THT:LED_D5.0mm-4_RGB, F.Cu at (76.9, 108.9)
- added D85: LED_RABG, LED_THT:LED_D5.0mm-4_RGB, F.Cu at (131.2, 108.8)
- added D86: LED_RABG, LED_THT:LED_D5.0mm-4_RGB, F.Cu at (177.3, 108.7)
- added D87: LED_RABG, LED_THT:LED_D5.0mm-4_RGB, F.Cu at (233.8, 108.8)
- added D88: LED_RABG, LED_THT:LED_D5.0mm-4_RGB, F.Cu at (285.3, 108.8)
- added D89: LED_RABG, LED_THT:LED_D5.0mm-4_RGB, F.Cu at (336.1, 108.9)
- added R1: 1.69kΩ, Resistor_SMD:R_0603_1608Metric_Pad1.05x0.95mm_HandSolder, F.Cu at (183.4, 173.6)
- added R11: 1k, Resistor_SMD:R_0603_1608Metric_Pad1.05x0.95mm_HandSolder, F.Cu at (357.6, 115.7)
- added R18: 20Ω, Resistor_SMD:R_0603_1608Metric_Pad1.05x0.95mm_HandSolder, F.Cu at (95.4, 168.2)
- added R19: 51Ω, Resistor_SMD:R_0603_1608Metric_Pad1.05x0.95mm_HandSolder, F.Cu at (143.4, 166.2)
- added R20: 20Ω, Resistor_SMD:R_0603_1608Metric_Pad1.05x0.95mm_HandSolder, F.Cu at (143.4, 162.7)
- added R21: 20Ω, Resistor_SMD:R_0603_1608Metric_Pad1.05x0.95mm_HandSolder, F.Cu at (143.4, 164.4)
- added R22: 51Ω, Resistor_SMD:R_0603_1608Metric_Pad1.05x0.95mm_HandSolder, B.Cu at (177.1, 170.7)
- added R23: 20Ω, Resistor_SMD:R_0603_1608Metric_Pad1.05x0.95mm_HandSolder, B.Cu at (175.4, 170.7)
- added R24: 20Ω, Resistor_SMD:R_0603_1608Metric_Pad1.05x0.95mm_HandSolder, B.Cu at (173.6, 170.7)
- added R25: 51Ω, Resistor_SMD:R_0603_1608Metric_Pad1.05x0.95mm_HandSolder, F.Cu at (222.4, 158.4)
- added R26: 20Ω, Resistor_SMD:R_0603_1608Metric_Pad1.05x0.95mm_HandSolder, F.Cu at (222.4, 161.9)
- added R27: 20Ω, Resistor_SMD:R_0603_1608Metric_Pad1.05x0.95mm_HandSolder, F.Cu at (222.4, 160.2)
- added R28: 51Ω, Resistor_SMD:R_0603_1608Metric_Pad1.05x0.95mm_HandSolder, B.Cu at (286.1, 168.9)
- added R29: 20Ω, Resistor_SMD:R_0603_1608Metric_Pad1.05x0.95mm_HandSolder, B.Cu at (289.6, 168.9)
- added R3: 10kΩ, Resistor_SMD:R_0603_1608Metric_Pad1.05x0.95mm_HandSolder, F.Cu at (254.0, 183.2)
- added R30: 20Ω, Resistor_SMD:R_0603_1608Metric_Pad1.05x0.95mm_HandSolder, B.Cu at (287.9, 168.9)
- added R31: 51Ω, Resistor_SMD:R_0603_1608Metric_Pad1.05x0.95mm_HandSolder, B.Cu at (336.1, 170.2)
- added R32: 20Ω, Resistor_SMD:R_0603_1608Metric_Pad1.05x0.95mm_HandSolder, B.Cu at (340.2, 170.2)
- added R33: 20Ω, Resistor_SMD:R_0603_1608Metric_Pad1.05x0.95mm_HandSolder, B.Cu at (338.6, 170.2)
- added R34: 100kΩ, Resistor_SMD:R_0603_1608Metric_Pad1.05x0.95mm_HandSolder, F.Cu at (234.9, 170.7)
- added R35: 10kΩ, Resistor_SMD:R_0603_1608Metric_Pad1.05x0.95mm_HandSolder, F.Cu at (198.6, 179.7)
- added R7: 2kΩ, Resistor_SMD:R_0603_1608Metric_Pad1.05x0.95mm_HandSolder, F.Cu at (241.1, 173.0)
- added REF**: 4-40_NPTH, QAZ:4-40_NPTH, F.Cu at (183.5, 127.3)
- added REF**: 4-40_NPTH, QAZ:4-40_NPTH, F.Cu at (321.5, 147.5)
- added REF**: 4-40_NPTH, QAZ:4-40_NPTH, F.Cu at (126.7, 147.5)
- added REF**: 4-40_NPTH, QAZ:4-40_NPTH, F.Cu at (104.5, 127.3)
- added REF**: 4-40_NPTH, QAZ:4-40_NPTH, F.Cu at (226.5, 147.5)
- added REF**: 4-40_NPTH, QAZ:4-40_NPTH, F.Cu at (278.5, 127.3)
- added SB15: SolderBridge, Resistor_SMD:R_0603_1608Metric_Pad1.05x0.95mm_HandSolder, F.Cu at (228.1, 161.9)
- added SB20: SolderBridge, Resistor_SMD:R_0603_1608Metric_Pad1.05x0.95mm_HandSolder, F.Cu at (222.4, 179.4)
- added SB21: SolderBridge, Resistor_SMD:R_0603_1608Metric_Pad1.05x0.95mm_HandSolder, F.Cu at (195.6, 172.4)
- added SB9: SolderBridge, Resistor_SMD:R_0603_1608Metric_Pad1.05x0.95mm_HandSolder, F.Cu at (219.1, 110.0)
- added TP10: TestPoint, QAZ:TestPoint_Thruhole_1.0mm, F.Cu at (251.6, 173.2)
- added TP11: TestPoint, QAZ:TestPoint_Thruhole_1.0mm, F.Cu at (253.4, 175.0)
- added TP14: TestPoint, QAZ:TestPoint_Thruhole_1.0mm, F.Cu at (248.2, 179.6)
- added TP15: TestPoint, QAZ:TestPoint_Thruhole_1.0mm, F.Cu at (257.4, 181.7)
- C1: value 100nF -> 4.7uF; footprint Capacitor_SMD:C_0603_1608Metric_Pad1.05x0.95mm_HandSolder -> Capacitor_SMD:C_0805_2012Metric_Pad1.15x1.40mm_HandSolder
- C10: renamed from C11; value 100nF -> 0.1uF
- C13: value 1uF -> 0.1uF
- C2: renamed from C3; value 100nF -> 0.1uF
- C4: renamed from C5; value 100nF -> 0.1uF
- C5: renamed from C6; value 100nF -> 0.1uF
- C8: renamed from C9; value 100nF -> 0.1uF
- R13: value 4.7k -> 1k
- R15: value 10k -> 5.1k
- R16: value 10k -> 51Ω
- R17: value 5.1k -> 20Ω; moved to F.Cu
- R2: value 10k -> 10kΩ
- R4: renamed from R10; value 1.3k -> 1.3kΩ
- R5: renamed from R11; value 1.3k -> 1.3kΩ
- R6: value 1k -> 10kΩ
- R8: value 1.69k -> 2kΩ
- R9: value 2.1k -> 5.1k
- SW1: value PTS525 -> JS102011SCQN; footprint QAZ:PTS525SM15 -> QAZ:JS102011SCQN_SPDT
- U3: value LP5009RUKR -> IS31FL3746A; footprint QAZ:QFN-20-1EP_3x3mm_P0.4mm_EP1.65x1.65mm_HS -> QAZ:QFN-32-1EP_4x4mm_P0.4mm_EP2.9x2.9mm_HS
- moved R12 160.5 mm to (359.1, 137.2)
- moved R16 158.8 mm to (95.4, 169.9)
- moved R17 141.1 mm to (95.4, 166.4), turned to 0 degrees
- moved SB5 124.6 mm to (108.6, 125.9), turned to 90 degrees
- moved R10 110.3 mm to (362.3, 96.7), turned to 0 degrees
- moved R9 104.0 mm to (214.2, 91.2)
- moved SB8 102.3 mm to (216.6, 108.3), turned to 0 degrees
- moved R13 95.7 mm to (350.4, 153.7)
- moved R14 94.0 mm to (291.0, 171.7), turned to 90 degrees
- moved TP1 84.2 mm to (190.6, 90.4)
- moved R5 83.9 mm to (263.6, 168.7)
- moved D3 80.4 mm to (263.6, 167.0), turned to 0 degrees
- moved C13 73.5 mm to (197.4, 176.1), turned to 90 degrees
- moved SB10 69.6 mm to (343.6, 182.4), turned to 270 degrees
- moved C12 67.8 mm to (195.6, 176.1), turned to 90 degrees
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- renumbered C10 to C9, D7 to D10, D8 to D11, D9 to D12, D10 to D13, D11 to D14, D12 to D15, D13 to D16, D14 to D17, D15 to D18, D16 to D19, LED5 to D2, D17 to D20, D18 to D21, D19 to D22, D20 to D23, D21 to D24, D22 to D25, D23 to D26, D24 to D27, D25 to D28, D26 to D29, LED6 to D3, D27 to D30, D28 to D31, D29 to D32, D30 to D33, D31 to D34, D32 to D35, D33 to D36, D34 to D37, D35 to D38, D36 to D39, D1 to D4, D37 to D40, D38 to D41, D40 to D43, D41 to D44, D42 to D45, D43 to D46, D44 to D47, D45 to D48, D46 to D49, D2 to D5, D47 to D50, D48 to D51, D49 to D52, D50 to D53, D51 to D54, D52 to D55, D53 to D56, D54 to D57, D55 to D58, D56 to D59, D3 to D6, D57 to D60, D58 to D61, D59 to D62, D60 to D63, D61 to D64, D62 to D65, D63 to D66, D64 to D67, D65 to D68, D66 to D69, D4 to D7, D67 to D70, D68 to D71, D5 to D8, D6 to D9, R3 to R10, R5 to R12, R7 to R14, SB2 to SB1, SB14 to SB10, SB15 to SB11, SB16 to SB12, SB17 to SB13, SB18 to SB14, SB20 to SB16, SB21 to SB17, SB22 to SB18, SB23 to SB19, SB7 to SB2, SB9 to SB3, SB10 to SB4, SB12 to SB6, SB13 to SB7, TP14 to TP12, TP15 to TP13, TP5 to TP4, TP6 to TP5, TP8 to TP6, TP10 to TP7, TP11 to TP8, TP12 to TP9
Connections:
- net /QAZ Testboard Keys/COL00 renamed /QAZ Keys/COL00
- net /QAZ Testboard Keys/COL01 renamed /QAZ Keys/COL01
- net /QAZ Testboard Keys/COL02 renamed /QAZ Keys/COL02
- net /QAZ Testboard Keys/COL03 renamed /QAZ Keys/COL03
- net /QAZ Testboard Keys/COL04 renamed /QAZ Keys/COL04
- net /QAZ Testboard Keys/COL05 renamed /QAZ Keys/COL05
- net /QAZ Testboard Keys/COL06 renamed /QAZ Keys/COL06
- net /QAZ Testboard Keys/COL07 renamed /QAZ Keys/COL07
- net /QAZ Testboard Keys/COL08 renamed /QAZ Keys/COL08
- net /QAZ Testboard Keys/COL09 renamed /QAZ Keys/COL09
- net /QAZ Testboard Keys/COL10 renamed /QAZ Keys/COL10
- net /QAZ Testboard Keys/COL11 renamed /QAZ Keys/COL11
- net /QAZ Testboard Keys/COL13 renamed /QAZ Keys/COL13
- net /QAZ Testboard Keys/COL14 renamed /QAZ Keys/COL14
- net /QAZ Testboard Keys/ROW00 renamed /QAZ Keys/ROW00
- net /QAZ Testboard Keys/ROW01 renamed /QAZ Keys/ROW01
- net /QAZ Testboard Keys/ROW02 renamed /QAZ Keys/ROW02
- net /QAZ Testboard Keys/ROW04 renamed /QAZ Keys/ROW04
- C1 pad 2: Net-(C1-Pad2) -> +5V
- C13 pad 2: Net-(C13-Pad2) -> Net-(C12-Pad2)
- C7 pad 1: Net-(C7-Pad1) -> /OSC_OUT
- CN1 pad A6: /QAZ External Connections/USB_D+ -> /USB_D+
- CN1 pad A7: /QAZ External Connections/USB_D- -> /USB_D-
- CN1 pad A8: Net-(CN1-PadA8) -> (no net)
- CN1 pad B6: /QAZ External Connections/USB_D+ -> /USB_D+
- CN1 pad B7: /QAZ External Connections/USB_D- -> /USB_D-
- CN1 pad B8: Net-(CN1-PadB8) -> (no net)
- D60 pad 1: /QAZ Testboard Keys/COL12 -> /QAZ Keys/COL12
- D61 pad 1: /QAZ Testboard Keys/COL12 -> /QAZ Keys/COL12
- R13 pad 1: /LED_SDA -> /QAZ Keys/ROW03
- R13 pad 2: +3V3 -> /ROW03
- R15 pad 1: /QAZ External Connections/SWDIO -> GND
- R15 pad 2: +3V3 -> Net-(CN1-PadB5)
- R16 pad 1: GND -> Net-(D72-Pad1)
- R16 pad 2: /QAZ External Connections/SWCLK -> /QAZ RGB/CS1
- R17 pad 1: GND -> Net-(D72-Pad4)
- R17 pad 2: Net-(CN1-PadB5) -> /QAZ RGB/CS2
- R2 pad 1: Net-(R2-Pad1) -> /SWDIO
- R2 pad 2: /BOOT0 -> +3V3
- R6 pad 1: /QAZ Testboard Keys/ROW03 -> Net-(R6-Pad1)
- R6 pad 2: /ROW03 -> /BOOT0
- R8 pad 1: Net-(LED4-Pad2) -> /LED_SDA
- R8 pad 2: +5V -> +3V3
- R9 pad 2: Net-(R9-Pad2) -> Net-(CN1-PadA5)
- SB5 pad 1: Net-(C7-Pad1) -> /COL12
- SB5 pad 2: /OSC_IN -> /QAZ Keys/COL12
- SB8 pad 1: Net-(LED3-Pad4) -> /USB_D+
- SB8 pad 2: +5V -> /USB_D_+
- SW1 pad 2: Net-(C1-Pad2) -> Net-(R6-Pad1)
- SW1 pad 3: (no net) -> +3V3
- SW10 pad 2: /QAZ Testboard Keys/ROW03 -> /QAZ Keys/ROW03
- SW15 pad 2: /QAZ Testboard Keys/ROW03 -> /QAZ Keys/ROW03
- SW20 pad 2: /QAZ Testboard Keys/ROW03 -> /QAZ Keys/ROW03
- SW24 pad 2: /QAZ Testboard Keys/ROW03 -> /QAZ Keys/ROW03
- SW28 pad 2: /QAZ Testboard Keys/ROW03 -> /QAZ Keys/ROW03
- SW33 pad 2: /QAZ Testboard Keys/ROW03 -> /QAZ Keys/ROW03
- SW37 pad 2: /QAZ Testboard Keys/ROW03 -> /QAZ Keys/ROW03
- SW41 pad 2: /QAZ Testboard Keys/ROW03 -> /QAZ Keys/ROW03
- SW46 pad 2: /QAZ Testboard Keys/ROW03 -> /QAZ Keys/ROW03
- SW5 pad 2: /QAZ Testboard Keys/ROW03 -> /QAZ Keys/ROW03
- SW51 pad 2: /QAZ Testboard Keys/ROW03 -> /QAZ Keys/ROW03
- SW56 pad 2: /QAZ Testboard Keys/ROW03 -> /QAZ Keys/ROW03
- SW63 pad 2: /QAZ Testboard Keys/ROW03 -> /QAZ Keys/ROW03
- SW68 pad 2: /QAZ Testboard Keys/ROW03 -> /QAZ Keys/ROW03
- TP12 pad 1: /USB_D- -> /USB_D_-
- TP13 pad 1: /USB_D+ -> /USB_D_+
- TP7 pad 1: /LED_EN -> /LED_SDB
- U1 pad 4: Net-(U1-Pad4) -> (no net)
- U2 pad 10: Net-(U2-Pad10) -> /ROW04
- U2 pad 11: Net-(U2-Pad11) -> /ROW00
- U2 pad 12: Net-(U2-Pad12) -> /ROW01
- U2 pad 13: Net-(U2-Pad13) -> /ROW02
- U2 pad 14: Net-(U2-Pad14) -> /ROW03
- U2 pad 15: /COL00 -> (no net)
- U2 pad 16: /COL01 -> (no net)
- U2 pad 17: /COL02 -> (no net)
- U2 pad 18: /ROW00 -> /HB_LED
- U2 pad 19: /ROW01 -> (no net)
- U2 pad 2: /COL11 -> /COL00
- U2 pad 20: /LED_EN -> /LED_SDB
- U2 pad 25: /ROW03 -> /COL03
- U2 pad 26: /COL03 -> /COL04
- U2 pad 27: /COL04 -> /COL05
- U2 pad 28: /COL05 -> /COL06
- U2 pad 3: /COL13 -> /COL01
- U2 pad 31: /COL06 -> /COL07
- U2 pad 32: /USB_D- -> /USB_D_-
- U2 pad 33: /USB_D+ -> /USB_D_+
- U2 pad 38: /ROW02 -> /COL08
- U2 pad 39: /HB_LED -> /COL09
- U2 pad 4: /COL14 -> /COL02
- U2 pad 40: /COL07 -> /COL10
- U2 pad 41: /ROW04 -> /COL11
- U2 pad 43: /COL08 -> /COL13
- U2 pad 45: /COL09 -> /COL14
- U2 pad 46: /COL10 -> (no net)
- U3 pad 1: Net-(C13-Pad2) -> /QAZ RGB/CS2
- U3 pad 10: Net-(SB40-Pad1) -> /QAZ RGB/CS10
- U3 pad 11: (no net) -> /QAZ RGB/CS11
- U3 pad 12: (no net) -> /QAZ RGB/CS12
- U3 pad 13: (no net) -> /QAZ RGB/CS13
- U3 pad 14: GND -> /QAZ RGB/CS14
- U3 pad 15: GND -> /QAZ RGB/CS15
- U3 pad 16: Net-(C12-Pad2) -> /QAZ RGB/CS16
- U3 pad 17: Net-(SB27-Pad2) -> /QAZ RGB/CS17
- U3 pad 18: Net-(SB28-Pad2) -> /QAZ RGB/CS18
- U3 pad 2: Net-(SB36-Pad1) -> /QAZ RGB/CS3
- U3 pad 20: Net-(R9-Pad2) -> /LED_SDB
- U3 pad 21: GND -> /LED_SCL
- U3 pad 3: Net-(SB35-Pad1) -> /QAZ RGB/CS4
- U3 pad 4: Net-(SB34-Pad1) -> /QAZ RGB/CS5
- U3 pad 5: Net-(SB39-Pad1) -> /QAZ RGB/CS6
- U3 pad 6: Net-(SB38-Pad1) -> /QAZ RGB/CS7
- U3 pad 7: Net-(SB37-Pad1) -> /QAZ RGB/CS8
- U3 pad 8: Net-(SB42-Pad1) -> /QAZ RGB/CS9
- U3 pad 9: Net-(SB41-Pad1) -> GND
- Y1 pad 1: Net-(C7-Pad1) -> /OSC_IN
- Y1 pad 2: Net-(C8-Pad1) -> /OSC_OUT
Routing:
- net /QAZ RGB/SW3: track 0.00 -> 448.6 mm, vias 0 -> 6
- net /QAZ RGB/SW2: track 0.00 -> 372.9 mm, vias 0 -> 3
- net /QAZ RGB/SW1: track 0.00 -> 321.1 mm, vias 0 -> 3
- net /QAZ Keys/ROW03: track 0.00 -> 283.6 mm, vias 0 -> 4
- net /QAZ Testboard Keys/ROW03: track 281.4 -> 0.00 mm, vias 4 -> 0
- net +5V: track 390.8 -> 139.9 mm
- net /RGB2_R: track 178.5 -> 0.00 mm, vias 6 -> 0
- net /RGB2_B: track 178.2 -> 0.00 mm, vias 6 -> 0
- net /RGB2_G: track 177.8 -> 0.00 mm, vias 6 -> 0
- net /QAZ RGB/CS16: track 0.00 -> 156.9 mm, vias 0 -> 1
- net /QAZ RGB/CS17: track 0.00 -> 156.8 mm, vias 0 -> 1
- net /QAZ RGB/CS18: track 0.00 -> 156.8 mm, vias 0 -> 1
- net /ROW01: track 6.70 -> 152.5 mm
- net +3V3: track 259.2 -> 123.0 mm, vias 2 -> 0
- net /USB_D_+: track 0.00 -> 128.2 mm
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- added copper zone on F.Cu, net GND
Other:
- outline, holes or cut-outs redrawn
- net class Default: clearance 0.1524 -> 0.127; trace_width 0.254 -> 0.25; via_dia 0.8 -> 0.5; via_drill 0.4 -> 0.25
- rule pad_to_mask_clearance: 0.05 -> 0.1
- rule trace_clearance: 0.1524 -> 0.127
- rule via_min_drill: 0.3 -> 0.2
- board text added: "+5V"
- board text added: "CLK"
- board text added: "DBG"
- board text added: "GND"
- board text added: "KB"
- board text added: "PG"
- board text added: "QAZ 65% v1.1"
- board text added: "SCL"
- board text added: "SDA"
- board text added: "SDB"
- board text added: "SWCLK"
- board text added: "SWDIO"
- board text added: "nRESET"
- board text removed: "APP"
- board text removed: "BOOT"
- board text removed: "QAZ 65% v1.1 - Anthony Needles"
- board text removed: "RESET"

Commit message: layers: added v2/v3 layers for qaz 65%
closes #4

v2 has slightly altered holes on the top of the outline, since the SWD
connector is not brought out.

v3 is for using a pcb as the plate layer (not sure if it will work..)
Parts:
- removed G***: LOGO, QAZ:qaz_logo_20mm
- moved R28 4.67 mm to (290.6, 170.2)
- moved R31 4.25 mm to (340.4, 170.2)
- moved R33 1.75 mm to (336.9, 170.2)
- moved R32 1.60 mm to (338.6, 170.2)
- moved R29 1.46 mm to (288.9, 170.2)
- moved R30 1.46 mm to (287.1, 170.2)
Connections:
- CN1 pad A8: (no net) -> Net-(CN1-PadA8)
- CN1 pad B8: (no net) -> Net-(CN1-PadB8)
- R16 pad 2: /QAZ RGB/CS1 -> /QAZ RGB/CS16
- R17 pad 2: /QAZ RGB/CS2 -> /QAZ RGB/CS17
- R18 pad 2: /QAZ RGB/CS3 -> /QAZ RGB/CS18
- R19 pad 2: /QAZ RGB/CS4 -> /QAZ RGB/CS13
- R20 pad 2: /QAZ RGB/CS5 -> /QAZ RGB/CS14
- R21 pad 2: /QAZ RGB/CS6 -> /QAZ RGB/CS15
- R22 pad 2: /QAZ RGB/CS7 -> /QAZ RGB/CS10
- R23 pad 2: /QAZ RGB/CS8 -> /QAZ RGB/CS11
- R24 pad 2: /QAZ RGB/CS9 -> /QAZ RGB/CS12
- R25 pad 2: /QAZ RGB/CS10 -> /QAZ RGB/CS7
- R26 pad 2: /QAZ RGB/CS11 -> /QAZ RGB/CS8
- R27 pad 2: /QAZ RGB/CS12 -> /QAZ RGB/CS9
- R28 pad 2: /QAZ RGB/CS13 -> /QAZ RGB/CS4
- R29 pad 2: /QAZ RGB/CS14 -> /QAZ RGB/CS5
- R30 pad 2: /QAZ RGB/CS15 -> /QAZ RGB/CS6
- R31 pad 2: /QAZ RGB/CS16 -> /QAZ RGB/CS1
- R32 pad 2: /QAZ RGB/CS17 -> /QAZ RGB/CS2
- R33 pad 2: /QAZ RGB/CS18 -> /QAZ RGB/CS3
- U1 pad 4: (no net) -> Net-(U1-Pad4)
- U2 pad 15: (no net) -> Net-(U2-Pad15)
- U2 pad 16: (no net) -> Net-(U2-Pad16)
- U2 pad 17: (no net) -> Net-(U2-Pad17)
- U2 pad 19: (no net) -> Net-(U2-Pad19)
- U2 pad 46: (no net) -> Net-(U2-Pad46)
- U3 pad 25: (no net) -> Net-(U3-Pad25)
Routing:
- net /QAZ RGB/CS1: track 125.6 -> 161.1 mm, vias 2 -> 1
- net /QAZ RGB/CS3: track 127.2 -> 158.5 mm, vias 2 -> 1
- net /QAZ RGB/CS2: track 126.9 -> 157.3 mm, vias 2 -> 1
- net /QAZ RGB/CS9: track 60.0 -> 32.3 mm, vias 1 -> 2
- net /QAZ RGB/CS8: track 58.1 -> 33.2 mm, vias 1 -> 2
- net /QAZ RGB/CS4: track 78.8 -> 101.9 mm, vias 2 -> 1
- net /QAZ RGB/CS5: track 78.9 -> 99.9 mm, vias 2 -> 1
- net /QAZ RGB/CS12: track 39.6 -> 57.7 mm, vias 2 -> 1
- net /QAZ RGB/CS6: track 80.9 -> 98.2 mm, vias 2 -> 1
- net /QAZ RGB/CS11: track 37.9 -> 54.2 mm, vias 2 -> 1
- net /QAZ RGB/CS7: track 54.4 -> 43.1 mm, vias 1 -> 2
- net /QAZ RGB/CS13: track 101.4 -> 92.0 mm, vias 1 -> 2
- net Net-(D76-Pad1): track 75.0 -> 83.9 mm
- net /QAZ RGB/CS16: track 156.9 -> 148.0 mm, vias 1 -> 2
- net Net-(D77-Pad1): track 72.7 -> 81.5 mm
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
Commit message: breakout: rgb conversion board
Made a conversion board for the LED driver conversion board. The RGB
LEDs chosen will not fit, and must be replaced in QAZ v1.1.
Parts:
- removed REF** (x6): 4-40_NPTH, QAZ:4-40_NPTH
- added H1: MountingHole, QAZ:4-40_NPTH, F.Cu at (104.5, 127.3)
- added H2: MountingHole, QAZ:4-40_NPTH, F.Cu at (226.5, 147.5)
- added H3: MountingHole, QAZ:4-40_NPTH, F.Cu at (126.7, 147.5)
- added H4: MountingHole, QAZ:4-40_NPTH, F.Cu at (278.5, 127.3)
- added H5: MountingHole, QAZ:4-40_NPTH, F.Cu at (183.5, 127.3)
- added H6: MountingHole, QAZ:4-40_NPTH, F.Cu at (321.5, 147.5)
- added JP1: Jumper_NC_Small, Connector_PinHeader_1.27mm:PinHeader_1x02_P1.27mm_Vertical, F.Cu at (184.0, 171.2)
- added JP2: Jumper_NC_Small, Connector_PinHeader_1.27mm:PinHeader_1x02_P1.27mm_Vertical, F.Cu at (184.0, 174.3)
- added JP3: Jumper_NC_Small, Connector_PinHeader_1.27mm:PinHeader_1x02_P1.27mm_Vertical, F.Cu at (268.1, 166.8)
- C14: value 1uF -> 0.1uF
- D72, D73, D74, D75, D76, D77, D78, D79, D80, D81, D82, D83, D84, D85, D86, D87, D88, D89: value LED_RABG -> 19-337C_RSBHGHC-A88_4T; footprint LED_THT:LED_D5.0mm-4_RGB -> QAZ:0606_1616Metric_HS
- R10, R11, R12, R13, R14: value 1k -> 1kΩ
- R15, R9: value 5.1k -> 5.1kΩ
- moved R1 3.92 mm to (180.8, 170.7), turned to 90 degrees
- moved D82 3.82 mm to (289.1, 142.2), turned to 180 degrees
- moved D88 3.82 mm to (289.1, 109.2), turned to 180 degrees
- moved D76 3.81 mm to (289.1, 165.4), turned to 180 degrees
- moved D83 3.36 mm to (339.4, 137.4), turned to 180 degrees
- moved D77 3.29 mm to (339.4, 165.4), turned to 180 degrees
- moved D89 3.26 mm to (339.4, 109.2), turned to 180 degrees
- moved D74 3.20 mm to (178.9, 162.9), turned to 180 degrees
- moved D1 3.00 mm to (179.1, 170.7), turned to 270 degrees
- moved R4 2.81 mm to (180.8, 174.4), turned to 270 degrees
- moved D75 2.24 mm to (235.9, 162.9), turned to 180 degrees
- moved D85 2.18 mm to (133.4, 109.2), turned to 180 degrees
- moved D73 2.16 mm to (133.4, 165.4), turned to 180 degrees
- moved D79 2.15 mm to (133.4, 130.4), turned to 180 degrees
- moved D87 2.08 mm to (235.9, 109.2), turned to 180 degrees
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Connections:
- D72 pad 4: Net-(D72-Pad4) -> /QAZ RGB/SW1
- D73 pad 4: Net-(D73-Pad4) -> /QAZ RGB/SW1
- D74 pad 4: Net-(D74-Pad4) -> /QAZ RGB/SW1
- D75 pad 4: Net-(D75-Pad4) -> /QAZ RGB/SW1
- D76 pad 4: Net-(D76-Pad4) -> /QAZ RGB/SW1
- D77 pad 4: Net-(D77-Pad4) -> /QAZ RGB/SW1
- D78 pad 4: Net-(D72-Pad4) -> /QAZ RGB/SW2
- D79 pad 4: Net-(D73-Pad4) -> /QAZ RGB/SW2
- D80 pad 4: Net-(D74-Pad4) -> /QAZ RGB/SW2
- D81 pad 4: Net-(D75-Pad4) -> /QAZ RGB/SW2
- D82 pad 4: Net-(D76-Pad4) -> /QAZ RGB/SW2
- D83 pad 4: Net-(D77-Pad4) -> /QAZ RGB/SW2
- D84 pad 4: Net-(D72-Pad4) -> /QAZ RGB/SW3
- D85 pad 4: Net-(D73-Pad4) -> /QAZ RGB/SW3
- D86 pad 4: Net-(D74-Pad4) -> /QAZ RGB/SW3
- D87 pad 4: Net-(D75-Pad4) -> /QAZ RGB/SW3
- D88 pad 4: Net-(D76-Pad4) -> /QAZ RGB/SW3
- D89 pad 4: Net-(D77-Pad4) -> /QAZ RGB/SW3
- R1 pad 2: +5V -> Net-(JP1-Pad2)
- R16 pad 1: Net-(D72-Pad1) -> Net-(D72-Pad3)
- R17 pad 1: Net-(D72-Pad4) -> Net-(D72-Pad1)
- R18 pad 1: Net-(D72-Pad3) -> Net-(D72-Pad5)
- R19 pad 1: Net-(D73-Pad1) -> Net-(D73-Pad3)
- R20 pad 1: Net-(D73-Pad4) -> Net-(D73-Pad1)
- R21 pad 1: Net-(D73-Pad3) -> Net-(D73-Pad5)
- R22 pad 1: Net-(D74-Pad1) -> Net-(D74-Pad3)
- R23 pad 1: Net-(D74-Pad4) -> Net-(D74-Pad1)
- R24 pad 1: Net-(D74-Pad3) -> Net-(D74-Pad5)
- R25 pad 1: Net-(D75-Pad1) -> Net-(D75-Pad3)
- R26 pad 1: Net-(D75-Pad4) -> Net-(D75-Pad1)
- R27 pad 1: Net-(D75-Pad3) -> Net-(D75-Pad5)
- R28 pad 1: Net-(D76-Pad1) -> Net-(D76-Pad3)
- R29 pad 1: Net-(D76-Pad4) -> Net-(D76-Pad1)
- R30 pad 1: Net-(D76-Pad3) -> Net-(D76-Pad5)
- R31 pad 1: Net-(D77-Pad1) -> Net-(D77-Pad3)
- R32 pad 1: Net-(D77-Pad4) -> Net-(D77-Pad1)
- R33 pad 1: Net-(D77-Pad3) -> Net-(D77-Pad5)
- R4 pad 2: +3V3 -> Net-(JP2-Pad2)
- R5 pad 2: /HB_LED -> Net-(JP3-Pad2)
Routing:
- net Net-(D73-Pad5): track 0.00 -> 104.4 mm
- net Net-(D74-Pad4): track 93.8 -> 0.00 mm
- net Net-(D73-Pad4): track 87.7 -> 0.00 mm
- net Net-(D75-Pad4): track 86.1 -> 0.00 mm
- net Net-(D72-Pad5): track 0.00 -> 85.2 mm
- net Net-(D75-Pad5): track 0.00 -> 84.4 mm
- net Net-(D74-Pad5): track 0.00 -> 84.3 mm, vias 0 -> 1
- net Net-(D76-Pad5): track 0.00 -> 82.1 mm, vias 0 -> 2
- net Net-(D77-Pad5): track 0.00 -> 79.9 mm, vias 0 -> 2
- net Net-(D76-Pad4): track 75.0 -> 0.00 mm
- net Net-(D72-Pad4): track 74.7 -> 0.00 mm
- net Net-(D77-Pad4): track 69.7 -> 0.00 mm
- net Net-(D74-Pad1): track 81.6 -> 96.7 mm, vias 0 -> 1
- net Net-(D74-Pad3): track 101.9 -> 87.5 mm, vias 0 -> 1
- net Net-(D73-Pad3): track 90.3 -> 104.4 mm
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Other:
- board text added: "D+"
- board text added: "D-"
- board text added: "DBG_TX"
- board text added: "USB"
- board text removed: "DBG"

Commit message: qaz 65% v1.2: in-progress, updated pcb
An issue seen with v1.1 (and v1.0 to a degree) was board warping. It's
suspected that a copper imbalance causes this, since there is a full
copper pour on the back of the board, and comparatively little copper on
the front of the board.

A ground pour was added to the top. This is desired over floating
copper, but requires many ground via to stitch the pour to ground, and
to prevent any antennae-like patches.

Also slightly moved some of the in-board screw holes so that they don't
brush up so close to key switches.
Parts:
- moved H6 2.24 mm to (323.5, 148.5)
- moved H3 1.12 mm to (126.2, 148.5)
Routing:
- net GND: track 115.8 -> 118.4 mm, vias 56 -> 160
Other:
- board text added: "QAZ 65% v1.2"
- board text removed: "QAZ 65% v1.1"
