File: hardware/QAZ_65/layers/plate_layer/plate_layer.kicad_pcb (KiCad board)
At the start: 2 copper layers, 326.8 x 117.3 mm, 0 parts

Commit message: qaz 65% v1.2: in-progress, updated pcb
An issue seen with v1.1 (and v1.0 to a degree) was board warping. It's
suspected that a copper imbalance causes this, since there is a full
copper pour on the back of the board, and comparatively little copper on
the front of the board.

A ground pour was added to the top. This is desired over floating
copper, but requires many ground via to stitch the pour to ground, and
to prevent any antennae-like patches.

Also slightly moved some of the in-board screw holes so that they don't
brush up so close to key switches.
Other:
- outline, holes or cut-outs redrawn
Changed lines of the file:
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@@
   )
   (page A3)
+  (title_block
+    (title "QAZ 65% Plate Layer")
+    (date 2021-08-29)
+    (rev v3)
+    (company "Anthony Needles")
+  )
   (layers
     (0 F.Cu signal)
@@
     (visible_elements 7FFFFFFF)
     (pcbplotparams
-      (layerselection 0x010fc_ffffffff)
+      (layerselection 0x010f0_ffffffff)
       (usegerberextensions false)
       (usegerberattributes false)
@@
       (drillshape 0)
       (scaleselection 1)
-      (outputdirectory ""))
+      (outputdirectory "plate_layer_out/"))
   )
   (net 0 "")
@@
   (gr_line (start 132.11227 197.973588) (end 131.67127 198.042588) (layer Edge.Cuts) (width 0.2))
   (gr_curve (pts (xy 198.639941 155.36055) (xy 198.907985 155.092507) (xy 199.05857 154.728962) (xy 199.05857 154.349891)) (layer Edge.Cuts) (width 0.2))
-  (gr_curve (pts (xy 101.199927 154.349891) (xy 101.199927 155.139263) (xy 101.839838 155.779176) (xy 102.62921 155.779177)) (layer Edge.Cuts) (width 0.2))
+  (gr_curve (pts (xy 99.199927 155.349891) (xy 99.199927 156.139263) (xy 99.839838 156.779176) (xy 100.62921 156.779177)) (layer Edge.Cuts) (width 0.2))
   (gr_line (start 133.26527 200.235588) (end 133.46727 199.838589) (layer Edge.Cuts) (width 0.2))
   (gr_line (start 50.73627 199.397588) (end 50.80627 199.838589) (layer Edge.Cuts) (width 0.2))
@@
   (gr_line (start 51.00927 200.235588) (end 51.32427 200.550588) (layer Edge.Cuts) (width 0.2))
   (gr_line (start 51.00927 198.560588) (end 50.80627 198.957588) (layer Edge.Cuts) (width 0.2))
-  (gr_curve (pts (xy 297.37914 155.779177) (xy 298.168511 155.779174) (xy 298.80842 155.139262) (xy 298.80842 154.349891)) (layer Edge.Cuts) (width 0.2))
-  (gr_curve (pts (xy 296.368479 155.36055) (xy 296.636523 155.628594) (xy 297.000069 155.779178) (xy 297.37914 155.779177)) (layer Edge.Cuts) (width 0.2))
-  (gr_curve (pts (xy 296.368479 153.339232) (xy 296.100435 153.607275) (xy 295.94985 153.97082) (xy 295.94985 154.349891)) (layer Edge.Cuts) (width 0.2))
+  (gr_curve (pts (xy 297.87914 156.779177) (xy 298.668511 156.779174) (xy 299.30842 156.139262) (xy 299.30842 155.349891)) (layer Edge.Cuts) (width 0.2))
+  (gr_curve (pts (xy 296.868479 156.36055) (xy 297.136523 156.628594) (xy 297.500069 156.779178) (xy 297.87914 156.779177)) (layer Edge.Cuts) (width 0.2))
+  (gr_curve (pts (xy 296.868479 154.339232) (xy 296.600435 154.607275) (xy 296.44985 154.97082) (xy 296.44985 155.349891)) (layer Edge.Cuts) (width 0.2))
   (gr_line (start 52.16127 197.973588) (end 51.720269 198.042588) (layer Edge.Cuts) (width 0.2))
   (gr_line (start 53.31427 200.235588) (end 53.51727 199.838589) (layer Edge.Cuts) (width 0.2))
   (gr_curve (pts (xy 321.05858 134.1) (xy 321.05858 133.720929) (xy 320.907995 133.357384) (xy 320.639951 133.089341)) (layer Edge.Cuts) (width 0.2))
-  (gr_curve (pts (xy 102.62921 155.779177) (xy 103.418582 155.779176) (xy 104.058493 155.139263) (xy 104.058493 154.349891)) (layer Edge.Cuts) (width 0.2))
+  (gr_curve (pts (xy 100.62921 156.779177) (xy 101.418582 156.779176) (xy 102.058493 156.139263) (xy 102.058493 155.349891)) (layer Edge.Cuts) (width 0.2))
   (gr_curve (pts (xy 147.05815 134.1) (xy 147.05815 133.310629) (xy 146.418241 132.670717) (xy 145.62887 132.670714)) (layer Edge.Cuts) (width 0.2))
-  (gr_curve (pts (xy 297.37914 152.920605) (xy 297.000069 152.920604) (xy 296.636523 153.071188) (xy 296.368479 153.339232)) (layer Edge.Cuts) (width 0.2))
+  (gr_curve (pts (xy 297.87914 153.920605) (xy 297.500069 153.920604) (xy 297.136523 154.071188) (xy 296.868479 154.339232)) (layer Edge.Cuts) (width 0.2))
   (gr_line (start 133.46727 198.957588) (end 133.26527 198.560588) (layer Edge.Cuts) (width 0.2))
   (gr_line (start 52.16127 200.822588) (end 52.60227 200.753588) (layer Edge.Cuts) (width 0.2))
@@
   (gr_line (start 51.32427 200.550588) (end 51.720269 200.753588) (layer Edge.Cuts) (width 0.2))
   (gr_line (start 50.80627 199.838589) (end 51.00927 200.235588) (layer Edge.Cuts) (width 0.2))
-  (gr_curve (pts (xy 295.94985 154.349891) (xy 295.94985 154.728962) (xy 296.100435 155.092507) (xy 296.368479 155.36055)) (layer Edge.Cuts) (width 0.2))
-  (gr_curve (pts (xy 102.62921 152.920605) (xy 101.839838 152.920606) (xy 101.199927 153.560519) (xy 101.199927 154.349891)) (layer Edge.Cuts) (width 0.2))
+  (gr_curve (pts (xy 296.44985 155.349891) (xy 296.44985 155.728962) (xy 296.600435 156.092507) (xy 296.868479 156.36055)) (layer Edge.Cuts) (width 0.2))
+  (gr_curve (pts (xy 100.62921 153.920605) (xy 99.839838 153.920606) (xy 99.199927 154.560519) (xy 99.199927 155.349891)) (layer Edge.Cuts) (width 0.2))
   (gr_line (start 50.80627 198.957588) (end 50.73627 199.397588) (layer Edge.Cuts) (width 0.2))
   (gr_line (start 51.32427 198.245588) (end 51.00927 198.560588) (layer Edge.Cuts) (width 0.2))
   (gr_line (start 53.51727 198.957588) (end 53.31427 198.560588) (layer Edge.Cuts) (width 0.2))
-  (gr_curve (pts (xy 298.80842 154.349891) (xy 298.80842 153.56052) (xy 298.168511 152.920608) (xy 297.37914 152.920605)) (layer Edge.Cuts) (width 0.2))
+  (gr_curve (pts (xy 299.30842 155.349891) (xy 299.30842 154.56052) (xy 298.668511 153.920608) (xy 297.87914 153.920605)) (layer Edge.Cuts) (width 0.2))
   (gr_curve (pts (xy 196.19999 154.349891) (xy 196.19999 154.728962) (xy 196.350575 155.092507) (xy 196.618619 155.36055)) (layer Edge.Cuts) (width 0.2))
-  (gr_curve (pts (xy 104.058493 154.349891) (xy 104.058493 153.560519) (xy 103.418582 152.920606) (xy 102.62921 152.920605)) (layer Edge.Cuts) (width 0.2))
+  (gr_curve (pts (xy 102.058493 155.349891) (xy 102.058493 154.560519) (xy 101.418582 153.920606) (xy 100.62921 153.920605)) (layer Edge.Cuts) (width 0.2))
   (gr_curve (pts (xy 144.19959 134.1) (xy 144.19959 134.889371) (xy 144.839499 135.529283) (xy 145.62887 135.529286)) (layer Edge.Cuts) (width 0.2))
   (gr_curve (pts (xy 240.6292 132.670714) (xy 240.250129 132.670713) (xy 239.886583 132.821297) (xy 239.618539 133.089341)) (layer Edge.Cuts) (width 0.2))
@@
   (gr_line (start 50.34927 202.873588) (end 50.19527 202.842588) (layer Edge.Cuts) (width 0.2))
   (gr_curve (pts (xy 318.2 134.1) (xy 318.2 134.479071) (xy 318.350585 134.842616) (xy 318.618629 135.110659)) (layer Edge.Cuts) (width 0.2))
-  (gr_text v3 (at 55.7 89.3) (layer F.SilkS)
+  (gr_text v3 (at 56.9 89.3) (layer F.SilkS)
     (effects (font (size 1.5 1.5) (thickness 0.3)))
   )
